Commit message: gazebo working

File: vacuscan_description/urdf/vacuscan_gazebo.urdf (robot description, URDF)
Before this commit: robot vacuscan_bot, 8 links, 7 joints
Joints:
- removed joint mount_left_link_to_mount_right_link_joint
- added joint rail_right_link_to_mount_right_link_joint: type prismatic, parent rail_right_link, child mount_right_link, origin xyz=0 0 0.06 rpy=0 0 0, axis 0 1 0, limit lower=-0.45 upper=0.2 effort=100 velocity=0.1, mimic joint=rail_left_link_to_mount_left_link_joint multiplier=1.0 offset=0.0
