Commit message: new urdf works, basic form only, no stl

File: vacuscan_description/urdf/vacuscan_rev0.urdf (robot description, URDF)
Before this commit: robot vacuscan_bot, 14 links, 13 joints
Links:
- removed link post_1_link
- removed link post_2_link
- removed link upper_base_link
- link base_link: geometry collision box size=0.8 1.0 0.1; visual box size=0.8 1.0 0.1
- link mount_center_link: geometry collision box size=0.2 0.02 0.1; visual box size=0.2 0.02 0.1
- link mount_left_link: geometry collision box size=0.1 0.1 0.02; visual box size=0.1 0.1 0.02
- link mount_right_link: geometry collision box size=0.1 0.1 0.02; visual box size=0.1 0.1 0.02
- link rail_center_link: geometry collision box size=1.1 0.1 0.1; visual box size=1.1 0.1 0.1
- link rail_left_link: geometry collision box size=0.1 1.0 0.1; visual box size=0.1 1.0 0.1
- link rail_right_link: geometry collision box size=0.1 1.0 0.1; visual box size=0.1 1.0 0.1
Joints:
- removed joint base_link_to_post_1_link_joint
- removed joint base_link_to_post_2_link_joint
- removed joint base_link_to_upper_link_joint
- joint base_link_to_rail_left_link_joint: origin xyz=0.3825 0 0.045 rpy=0 0 0 -> xyz=0.5 0 0.0 rpy=0 0 0
- joint base_link_to_rail_right_link_joint: origin xyz=-0.3825 0 0.045 rpy=0 0 0 -> xyz=-0.5 0 0.0 rpy=0 0 0
- joint camera2_joint: origin xyz=-0.8 0.05 0.8 rpy=0 0.785 0 -> xyz=-0.8 0.25 0.8 rpy=0 0.785 0
- joint camera_joint: origin xyz=0.0 0.05 1.2 rpy=0 1.57 0 -> xyz=0.0 0.25 1.2 rpy=0 1.57 0
- joint laser_joint: origin xyz=0.0 0.05 1.5 rpy=1.57 0 0 -> xyz=0.0 0.25 1.5 rpy=1.57 0 0
- joint mount_center_link_to_wafer_holder_link_joint: origin xyz=0 0.245 -0.09 rpy=0 0 0 -> xyz=0 0.2 -0.045 rpy=0 0 0
- joint mount_left_link_to_mount_right_link_joint: origin xyz=-0.765 0 0 rpy=0 0 0 -> xyz=-1.0 0 0 rpy=0 0 0
- joint mount_left_link_to_rail_center_link_joint: origin xyz=-0.3825 0 0.045 rpy=0 0 0 -> xyz=-0.5 0 0.06 rpy=0 0 0
- joint x_control_joint: origin xyz=0 0 0.045 rpy=0 0 0 -> xyz=0 0.06 0 rpy=0 0 0
- joint y_control_joint: origin xyz=0 -0.20 0.045 rpy=0 0 0 -> xyz=0 0 0.06 rpy=0 0 0
